Commit message: Working on fixing urdf errors

File: droplet_description/pf400_description/urdf/droplet.urdf (robot description, URDF)
Before this commit: robot Droplet_Setup, 1 links, 1 joints
Links:
- link droplet_base: geometry visual mesh filename=package://droplet_description/meshes/droplet_base.stl scale=0.02 0.02 0.02
Joints:
- removed joint rail_link
